Commit message: 20241226_alpha_1.1.0

File: urdf/arx5_description_ik.urdf (robot description, URDF)
Before this commit: robot arx5_description, 6 links, 5 joints
Links:
- added link fl_link6, mass 0.462244960775882; collision mesh filename=package://arx5p2/meshes/link6.STL; visual mesh filename=package://arx5p2/meshes/link6.STL
Joints:
- added joint fl_joint6: type revolute, parent fl_link5, child fl_link6, origin xyz=0.02845 0 0.0825 rpy=-3.1416 0 0, axis 1 0 0, limit lower=-10 upper=10 effort=100 velocity=1000

Commit message: 20250320压板操作最终版

File: urdf/arx5_description_ik.urdf (robot description, URDF)
Before this commit: robot arx5_description, 7 links, 6 joints
Joints:
- joint fl_joint2: limit lower=-0.05 upper=10 effort=100 velocity=1000 -> lower=-0.05 upper=3.2 effort=100 velocity=1000
- joint fl_joint3: limit lower=-0.05 upper=10 effort=100 velocity=1000 -> lower=-0.05 upper=3.2 effort=100 velocity=1000
